Commit message: change the urdf

File: catkin_ws/src/iiwa_tool/iiwa_tool_description/urdf/iiwa14_tool.urdf.xacro (robot description, xacro)
@@ -6,6 +6,4 @@
   <!--Import the iiwa14 macro -->
   <xacro:include filename="$(find iiwa_description)/urdf/iiwa14.xacro"/>
-  <!--Import the ez gripper files-->
-  <xacro:include filename="$(find iiwa_tool_description)/urdf/fusg_articulated.urdf.xacro"/>
   <!--  Arguments for the iiwa14 macro  -->
   <xacro:arg name="hardware_interface" default="PositionJointInterface"/>
@@ -84,10 +82,10 @@
     </inertial>
   </link>
-  <joint name="table_joint" type="fixed">
+  <joint name="conveyor_joint" type="fixed">
     <parent link="world"/>
-    <child link = "table"/>
-    <origin xyz="0.6 0.6 0" rpy="0 0 0"/>
-  </joint>
-  <link name="table">
+    <child link = "conveyor"/>
+    <origin xyz="0.6 1.7 0" rpy="0 0 0"/>
+  </joint>
+  <link name="conveyor">
     <visual>
       <origin xyz="0 0 0" rpy="0 0 0"/>
@@ -119,30 +117,25 @@
     </inertial>
   </link>
-  <joint name="camera_unit_joint" type="fixed">
-    <parent link="table"/>
-    <child link = "camera_unit"/>
-    <origin xyz="0.22 0.65 0.9" rpy="0 0 3.14"/>
-  </joint>
-  <link name="camera_unit">
-    <visual>
-      <origin xyz="0 0 0" rpy="0 0 0"/>
-      <geometry>
-        <mesh filename="package://iiwa_tool_description/meshes/visual/camera_unit_simple.dae"/>
-      </geometry>
-    </visual>
-    <collision>
-      <origin xyz="0 0 0" rpy="0 0 0"/>
-      <geometry>
-        <mesh filename="package://iiwa_tool_description/meshes/collision/camera_unit_simple.stl"/>
-      </geometry>
-    </collision>
-<!--
-    <collision>
-      <origin xyz="0 0 0" rpy="0 0 0"/>
-      <geometry>
-        <box size="0.1 0.1 0.1"/>
-      </geometry>
-    </collision>
--->
+  <joint name="round_table_joint" type="fixed">
+    <parent link="world"/>
+    <child link = "round_table"/>
+    <origin xyz="0 -0.7 0.485" rpy="0 0 0"/>
+  </joint>
+  <link name="round_table">
+    <visual>
+      <origin xyz="0 0 0" rpy="0 0 0"/>
+      <geometry>
+        <cylinder length="0.05" radius="0.43"/>
+      </geometry>
+      <material name="green">
+        <color rgba="0.0 0.8 0.0 0.5"/>
+      </material>
+    </visual>
+    <collision>
+      <origin xyz="0 0 0" rpy="0 0 0"/>
+      <geometry>
+        <cylinder length="0.05" radius="0.43"/>
+      </geometry>
+    </collision>
     <inertial>
       <origin xyz="0 0 1" rpy="0 0 0"/>
@@ -155,7 +148,7 @@
   </link>
   <joint name="heater_unit_joint" type="fixed">
-    <parent link="table"/>
+    <parent link="conveyor"/>
     <child link = "heater_unit"/>
-    <origin xyz="0.22 0.5 0.9" rpy="0 0 3.14"/>
+    <origin xyz="0.242 -1.4 0.8" rpy="0 0 1.57"/>
   </joint>
   <link name="heater_unit">
@@ -163,18 +156,21 @@
       <origin xyz="0 0 0" rpy="0 0 0"/>
       <geometry>
-        <mesh filename="package://iiwa_tool_description/meshes/visual/heater_unit_simple.dae"/>
-      </geometry>
-    </visual>
-    <collision>
-      <origin xyz="0 0 0" rpy="0 0 0"/>
-      <geometry>
-        <mesh filename="package://iiwa_tool_description/meshes/collision/heater_unit_simple.stl"/>
-      </geometry>
-    </collision>
-<!--
-    <collision>
-      <origin xyz="0 0 0" rpy="0 0 0"/>
-      <geometry>
-        <box size="0.1 0.1 0.1"/>
+        <mesh filename="package://iiwa_tool_description/meshes/visual/heater_unit.stl"/>
+      </geometry>
+      <material name="gray">
+        <color rgba="0.7 0.7 0.7 0.2"/>
+      </material>
+    </visual>
+    <collision>
+      <origin xyz="0 0.25 0.32" rpy="0 0 0"/>
+      <geometry>
+        <box size="0.22 0.445 0.4"/>
+      </geometry>
+    </collision>
+<!--
+    <collision>
+      <origin xyz="0 0 0" rpy="0 0 0"/>
+      <geometry>
+        <mesh filename="package://iiwa_tool_description/meshes/collision/heater_unit.stl"/>
       </geometry>
     </collision>
@@ -194,8 +190,69 @@
   </xacro:iiwa14>
   <!-- Add the gripper. Called from the file imported at the top of this code.-->
-  <softmatics_gripper prefix="tool" parent_link="iiwa_link_ee">
-    <origin xyz="0 0 0" rpy="0 0 ${PI/2}"/>
-  </softmatics_gripper>
-  <!--  Here we define another dummy joint. It is placed at the end of the tool, so we can then attach a frame at its TCP for control -->
+  <link name="tool_mount">
+    <visual>
+      <origin xyz="0 0 0" rpy="0 ${-pi/2} ${pi/2}"/>
+      <geometry>
+        <mesh filename="package://iiwa_tool_description/meshes/visual/iiwa_tool_mount.stl"/>
+      </geometry>
+      <material name="">
+        <color rgba="0.8 0.8 0.8 1"/>
+      </material>
+    </visual>
+    <collision>
+      <origin xyz="0 0 0" rpy="0 ${-pi/2} ${pi/2}"/>
+      <geometry>
+        <mesh filename="package://iiwa_tool_description/meshes/collision/iiwa_tool_mount.stl"/>
+      </geometry>
+    </collision>
+  </link>
+  <joint name="eef_base_joint" type="fixed">
+    <origin xyz="0 0 0.0095" rpy="0 0 0"/>
+    <parent link="tool_mount"/>
+    <child link="eef_base"/>
+  </joint>
+  <link name="eef_base">
+    <visual>
+      <origin xyz="0 0 0" rpy="0 0 0"/>
+      <geometry>
+        <mesh filename="package://iiwa_tool_description/meshes/visual/hande_base.stl"/>
+      </geometry>
+      <material name="">
+        <color rgba="0.8 0.8 0.8 1"/>
+      </material>
+    </visual>
+    <collision>
+      <origin xyz="0 0 0" rpy="0 0 0"/>
+      <geometry>
+        <mesh filename="package://iiwa_tool_description/meshes/collision/hande_base.stl"/>
+      </geometry>
+    </collision>
+  </link>
+  <joint name="eef_joint" type="fixed">
+    <origin xyz="0 0 0.0015" rpy="0 0 0"/>
+    <parent link="eef_base"/>
+    <child link="eef"/>
+  </joint>
+  <link name="eef">
+    <visual>
+      <origin xyz="0 0 0" rpy="0 0 0"/>
+      <geometry>
+        <mesh filename="package://iiwa_tool_description/meshes/visual/hande.stl"/>
+      </geometry>
+      <material name="">
+        <color rgba="0.8 0.8 0.8 1"/>
+      </material>
+    </visual>
+    <collision>
+      <geometry>
+        <mesh filename="package://iiwa_tool_description/meshes/collision/hande.stl"/>
+      </geometry>
+    </collision>
+  </link>
+  <joint name="tool_joint" type="fixed">
+    <parent link="iiwa_link_ee"/>
+    <child link="tool_mount"/>
+    <origin xyz="0 0 0.001" rpy="0 0 ${PI/2}"/>
+  </joint>
   <joint name="tool_tip_joint" type="fixed">
     <parent link="iiwa_link_ee"/>

Commit message: add workspace in the simulation

File: catkin_ws/src/iiwa_tool/iiwa_tool_description/urdf/iiwa14_tool.urdf.xacro (robot description, xacro)
@@ -31,12 +31,4 @@
       </geometry>
     </collision>
-<!--
-    <collision>
-      <origin xyz="0 0 0" rpy="0 0 0"/>
-      <geometry>
-        <mesh filename="package://iiwa_tool_description/meshes/collision/base.stl"/>
-      </geometry>
-    </collision>
--->
     <inertial>
       <origin xyz="0 0 1" rpy="0 0 0"/>
@@ -65,12 +57,4 @@
       </geometry>
     </collision>
-<!--
-    <collision>
-      <origin xyz="0 0 0.12" rpy="0 0 0"/>
-      <geometry>
-        <mesh filename="package://iiwa_tool_description/meshes/collision/mount.stl"/>
-      </geometry>
-    </collision>
--->
     <inertial>
       <origin xyz="0 0 1" rpy="0 0 0"/>
@@ -100,12 +84,64 @@
       </geometry>
     </collision>
-<!--
-    <collision>
-      <origin xyz="0 0 0" rpy="0 0 0"/>
-      <geometry>
-        <mesh filename="package://iiwa_tool_description/meshes/collision/conveyor.stl"/>
-      </geometry>
-    </collision>
--->
+    <inertial>
+      <origin xyz="0 0 1" rpy="0 0 0"/>
+      <mass value="1"/>
+      <inertia
+        ixx="1.0" ixy="0.0" ixz="0.0"
+        iyy="1.0" iyz="0.0"
+        izz="1.0"/>
+    </inertial>
+  </link>
+  <joint name="tv_joint" type="fixed">
+    <parent link="world"/>
+    <child link = "tv"/>
+    <origin xyz="0.6 -0.9 1.9" rpy="-0.1745 0 0.78"/>
+  </joint>
+  <link name="tv">
+    <visual>
+      <origin xyz="0 0 0" rpy="0 0 0"/>
+      <geometry>
+        <box size="1.1 0.1 0.6"/>
+      </geometry>
+      <material name="gray">
+        <color rgba="0.7 0.7 0.7 0.2"/>
+      </material>
+    </visual>
+    <collision>
+      <origin xyz="0 0 0" rpy="0 0 0"/>
+      <geometry>
+        <box size="1.1 0.1 0.6"/>
+      </geometry>
+    </collision>
+    <inertial>
+      <origin xyz="0 0 1" rpy="0 0 0"/>
+      <mass value="1"/>
+      <inertia
+        ixx="1.0" ixy="0.0" ixz="0.0"
+        iyy="1.0" iyz="0.0"
+        izz="1.0"/>
+    </inertial>
+  </link>
+  <joint name="frame_joint" type="fixed">
+    <parent link="world"/>
+    <child link = "frame"/>
+    <origin xyz="-0.2 0.8 0.9" rpy="0 0 0"/>
+  </joint>
+  <link name="frame">
+    <visual>
+      <origin xyz="0 0 0" rpy="0 0 0"/>
+      <geometry>
+        <mesh filename="package://iiwa_tool_description/meshes/visual/workspace.stl"/>
+      </geometry>
+      <material name="gray">
+        <color rgba="0.7 0.7 0.7 0.2"/>
+      </material>
+    </visual>
+    <collision>
+      <origin xyz="0 0 -0.5" rpy="0 0 0"/>
+      <geometry>
+        <box size="1.0 1.0 0.8"/>
+      </geometry>
+    </collision>
     <inertial>
       <origin xyz="0 0 1" rpy="0 0 0"/>
@@ -168,12 +204,4 @@
       </geometry>
     </collision>
-<!--
-    <collision>
-      <origin xyz="0 0 0" rpy="0 0 0"/>
-      <geometry>
-        <mesh filename="package://iiwa_tool_description/meshes/collision/heater_unit.stl"/>
-      </geometry>
-    </collision>
--->
     <inertial>
       <origin xyz="0 0 1" rpy="0 0 0"/>

Commit message: add iiwa_hande in the simulation

File: catkin_ws/src/iiwa_tool/iiwa_tool_description/urdf/iiwa14_tool.urdf.xacro (robot description, xacro)
@@ -153,4 +153,34 @@
     </inertial>
   </link>
+  <joint name="iiwa2_joint" type="fixed">
+    <parent link="frame"/>
+    <child link = "iiwa2"/>
+    <origin xyz="0.35 0 0" rpy="1.57 0 0"/>
+  </joint>
+  <link name="iiwa2">
+    <visual>
+      <origin xyz="0 0 0" rpy="0 0 0"/>
+      <geometry>
+        <mesh filename="package://iiwa_tool_description/meshes/visual/iiwa_hande.stl"/>
+      </geometry>
+      <material name="gray">
+        <color rgba="0.7 0.7 0.7 0.2"/>
+      </material>
+    </visual>
+    <collision>
+      <origin xyz="0 0.8 0" rpy="0 0 0"/>
+      <geometry>
+        <box size="0.2 1.6 0.2"/>
+      </geometry>
+    </collision>
+    <inertial>
+      <origin xyz="0 0 1" rpy="0 0 0"/>
+      <mass value="1"/>
+      <inertia
+        ixx="1.0" ixy="0.0" ixz="0.0"
+        iyy="1.0" iyz="0.0"
+        izz="1.0"/>
+    </inertial>
+  </link>
   <joint name="round_table_joint" type="fixed">
     <parent link="world"/>

Commit message: correct the iiwa2's pose and change the mesh

File: catkin_ws/src/iiwa_tool/iiwa_tool_description/urdf/iiwa14_tool.urdf.xacro (robot description, xacro)
@@ -156,5 +156,5 @@
     <parent link="frame"/>
     <child link = "iiwa2"/>
-    <origin xyz="0.35 0 0" rpy="1.57 0 0"/>
+    <origin xyz="0.30 0.34 0" rpy="1.57 0 0"/>
   </joint>
   <link name="iiwa2">
@@ -171,5 +171,5 @@
       <origin xyz="0 0.8 0" rpy="0 0 0"/>
       <geometry>
-        <box size="0.2 1.6 0.2"/>
+        <box size="0.25 1.5 0.25"/>
       </geometry>
     </collision>

Commit message: add softjig

File: catkin_ws/src/iiwa_tool/iiwa_tool_description/urdf/iiwa14_tool.urdf.xacro (robot description, xacro)
@@ -183,4 +183,34 @@
     </inertial>
   </link>
+  <joint name="softjig_joint" type="fixed">
+    <parent link="frame"/>
+    <child link = "softjig"/>
+    <origin xyz="0.45 0 0" rpy="1.57 0 3.14"/>
+  </joint>
+  <link name="softjig">
+    <visual>
+      <origin xyz="0 0 0" rpy="0 0 0"/>
+      <geometry>
+        <mesh filename="package://iiwa_tool_description/meshes/visual/softjig.stl"/>
+      </geometry>
+      <material name="gray_dark">
+        <color rgba="0.7 0.7 0.7 1.0"/>
+      </material>
+    </visual>
+    <collision>
+      <origin xyz="0 0 0" rpy="0 0 0"/>
+      <geometry>
+        <mesh filename="package://iiwa_tool_description/meshes/collision/softjig.stl"/>
+      </geometry>
+    </collision>
+    <inertial>
+      <origin xyz="0 0 1" rpy="0 0 0"/>
+      <mass value="1"/>
+      <inertia
+        ixx="1.0" ixy="0.0" ixz="0.0"
+        iyy="1.0" iyz="0.0"
+        izz="1.0"/>
+    </inertial>
+  </link>
   <joint name="round_table_joint" type="fixed">
     <parent link="world"/>

Commit message: delete unnecessary files and change some precise collision models to primitive shapes

File: catkin_ws/src/iiwa_tool/iiwa_tool_description/urdf/iiwa14_tool.urdf.xacro (robot description, xacro)
@@ -289,7 +289,7 @@
     </visual>
     <collision>
-      <origin xyz="0 0 0" rpy="0 ${-pi/2} ${pi/2}"/>
-      <geometry>
-        <mesh filename="package://iiwa_tool_description/meshes/collision/iiwa_tool_mount.stl"/>
+      <origin xyz="0 0 0.001" rpy="0 0 0"/>
+      <geometry>
+        <cylinder length="0.016" radius="0.038"/>
       </geometry>
     </collision>
@@ -311,7 +311,7 @@
     </visual>
     <collision>
-      <origin xyz="0 0 0" rpy="0 0 0"/>
-      <geometry>
-        <mesh filename="package://iiwa_tool_description/meshes/collision/hande_base.stl"/>
+      <origin xyz="0 0 0.0095" rpy="0 0 0"/>
+      <geometry>
+        <cylinder length="0.022" radius="0.038"/>
       </geometry>
     </collision>

Commit message: correct orientations

File: catkin_ws/src/iiwa_tool/iiwa_tool_description/urdf/iiwa14_tool.urdf.xacro (robot description, xacro)
@@ -275,5 +275,5 @@
   <!-- Here we insert an iiwa14 robot in the scene, it's origin is just on top of the box previously defined. You can use 0,0,0 if you don't have that. -->
   <xacro:iiwa14 hardware_interface="$(arg hardware_interface)" robot_name="$(arg robot_name)" parent="mount">
-    <origin xyz="0 0 0.978" rpy="0 0 0"/>
+    <origin xyz="0 0 0.978" rpy="0 0 3.14"/>
   </xacro:iiwa14>
   <!-- Add the gripper. Called from the file imported at the top of this code.-->
@@ -318,5 +318,5 @@
   </link>
   <joint name="eef_joint" type="fixed">
-    <origin xyz="0 0 0.0015" rpy="0 0 0"/>
+    <origin xyz="0 0 0.0015" rpy="0 0 3.14"/>
     <parent link="eef_base"/>
     <child link="eef"/>

Commit message: modify collision models

File: catkin_ws/src/iiwa_tool/iiwa_tool_description/urdf/iiwa14_tool.urdf.xacro (robot description, xacro)
@@ -289,7 +289,7 @@
     </visual>
     <collision>
-      <origin xyz="0 0 0.001" rpy="0 0 0"/>
-      <geometry>
-        <cylinder length="0.016" radius="0.038"/>
+      <origin xyz="0 0 0.005" rpy="0 0 0"/>
+      <geometry>
+        <cylinder length="0.006" radius="0.038"/>
       </geometry>
     </collision>
@@ -313,5 +313,5 @@
       <origin xyz="0 0 0.0095" rpy="0 0 0"/>
       <geometry>
-        <cylinder length="0.022" radius="0.038"/>
+        <cylinder length="0.020" radius="0.038"/>
       </geometry>
     </collision>

Commit message: correct simulation environment

File: catkin_ws/src/iiwa_tool/iiwa_tool_description/urdf/iiwa14_tool.urdf.xacro (robot description, xacro)
@@ -24,4 +24,7 @@
         <mesh filename="package://iiwa_tool_description/meshes/visual/base.dae"/>
       </geometry>
+      <material name="gray">
+        <color rgba="0.7 0.7 0.7 0.2"/>
+      </material>
     </visual>
     <collision>
@@ -43,4 +46,5 @@
     <parent link="base"/>
     <child link="mount"/>
+    <origin xyz="0 0 0" rpy="0 0 -1.57"/>
   </joint>
   <link name="mount">
@@ -48,6 +52,9 @@
       <origin xyz="0 0 0.145" rpy="0 0 0"/>
       <geometry>
-        <mesh filename="package://iiwa_tool_description/meshes/visual/mount.dae"/>
-      </geometry>
+        <mesh filename="package://iiwa_tool_description/meshes/visual/mount.stl"/>
+      </geometry>
+      <material name="gray">
+        <color rgba="0.7 0.7 0.7 0.2"/>
+      </material>
     </visual>
     <collision>
@@ -77,4 +84,7 @@
         <mesh filename="package://iiwa_tool_description/meshes/visual/conveyor.dae"/>
       </geometry>
+      <material name="gray">
+        <color rgba="0.7 0.7 0.7 0.2"/>
+      </material>
     </visual>
     <collision>
@@ -126,5 +136,5 @@
     <parent link="world"/>
     <child link = "frame"/>
-    <origin xyz="-0.2 0.8 0.9" rpy="0 0 0"/>
+    <origin xyz="-0.2 0.8 0.84" rpy="0 0 0"/>
   </joint>
   <link name="frame">
@@ -139,22 +149,44 @@
     </visual>
     <collision>
-      <origin xyz="0 0 -0.5" rpy="0 0 0"/>
-      <geometry>
-        <box size="1.0 1.0 0.8"/>
-      </geometry>
-    </collision>
-    <inertial>
-      <origin xyz="0 0 1" rpy="0 0 0"/>
-      <mass value="1"/>
-      <inertia
-        ixx="1.0" ixy="0.0" ixz="0.0"
-        iyy="1.0" iyz="0.0"
-        izz="1.0"/>
-    </inertial>
+      <origin xyz="0 0 -0.4" rpy="0 0 0"/>
+      <geometry>
+        <box size="1.0 1.0 0.7"/>
+      </geometry>
+    </collision>
+    <inertial>
+      <origin xyz="0 0 1" rpy="0 0 0"/>
+      <mass value="1"/>
+      <inertia
+        ixx="1.0" ixy="0.0" ixz="0.0"
+        iyy="1.0" iyz="0.0"
+        izz="1.0"/>
+    </inertial>
+  </link>
+  <joint name="workspace_mount_joint" type="fixed">
+      <origin xyz="0.30 0.34 0.016" rpy="0 0 0"/>
+      <parent link="frame"/>
+      <child link="workspace_mount"/>
+  </joint>
+  <link name="workspace_mount">
+      <visual>
+          <origin xyz="0 0 0" rpy="0 0 0"/>
+          <geometry>
+              <box size="0.3 0.3 0.03"/>
+          </geometry>
+          <material name="gray">
+              <color rgba="0.7 0.7 0.7 0.2"/>
+          </material>
+      </visual>
+      <collision>
+          <origin xyz="0 0 0" rpy="0 0 0"/>
+          <geometry>
+              <box size="0.3 0.3 0.03"/>
+          </geometry>
+      </collision>
   </link>
   <joint name="iiwa2_joint" type="fixed">
-    <parent link="frame"/>
+    <parent link="workspace_mount"/>
     <child link = "iiwa2"/>
-    <origin xyz="0.30 0.34 0" rpy="1.57 0 0"/>
+    <origin xyz="0 0 0" rpy="1.57 0 0.785398"/>
   </joint>
   <link name="iiwa2">
@@ -194,5 +226,5 @@
         <mesh filename="package://iiwa_tool_description/meshes/visual/softjig.stl"/>
       </geometry>
-      <material name="gray_dark">
+      <material name="dark_gray">
         <color rgba="0.7 0.7 0.7 1.0"/>
       </material>
@@ -216,5 +248,5 @@
     <parent link="world"/>
     <child link = "round_table"/>
-    <origin xyz="0 -0.7 0.485" rpy="0 0 0"/>
+    <origin xyz="0 -0.7 0.55" rpy="0 0 0"/>
   </joint>
   <link name="round_table">
@@ -275,5 +307,5 @@
   <!-- Here we insert an iiwa14 robot in the scene, it's origin is just on top of the box previously defined. You can use 0,0,0 if you don't have that. -->
   <xacro:iiwa14 hardware_interface="$(arg hardware_interface)" robot_name="$(arg robot_name)" parent="mount">
-    <origin xyz="0 0 0.978" rpy="0 0 3.14"/>
+    <origin xyz="0 0 0.972" rpy="0 0 -1.57"/>
   </xacro:iiwa14>
   <!-- Add the gripper. Called from the file imported at the top of this code.-->
