Commit message: save

File: catkin_ws/src/iiwa_tool/iiwa_tool_description/urdf/iiwa14_tool.urdf.xacro (robot description, xacro)
@@ -9,70 +9,11 @@
   <xacro:arg name="hardware_interface" default="PositionJointInterface"/>
   <xacro:arg name="robot_name" default="iiwa"/>
+  <link name="$(arg robot_name)_floating_link" />
   <!--  Define the 3D space -->
-  <link name="world"/>
-  <gazebo reference="world">
+  <gazebo reference="$(arg robot_name)_floating_link">
     <static>true</static>
   </gazebo>
-  <joint name="base_joint" type="fixed">
-    <parent link="world"/>
-    <child link="base"/>
-  </joint>
-  <link name="base">
-    <visual>
-      <origin xyz="0 0 0" rpy="0 0 0"/>
-      <geometry>
-        <mesh filename="package://iiwa_tool_description/meshes/visual/base.dae"/>
-      </geometry>
-      <material name="gray">
-        <color rgba="0.7 0.7 0.7 0.2"/>
-      </material>
-    </visual>
-    <collision>
-      <origin xyz="0 0 0.06" rpy="0 0 0"/>
-      <geometry>
-        <box size="0.4 0.4 0.10"/>
-      </geometry>
-    </collision>
-    <inertial>
-      <origin xyz="0 0 1" rpy="0 0 0"/>
-      <mass value="1"/>
-      <inertia
-        ixx="1.0" ixy="0.0" ixz="0.0"
-        iyy="1.0" iyz="0.0"
-        izz="1.0"/>
-    </inertial>
-  </link>
-  <joint name="mount_joint" type="fixed">
-    <parent link="base"/>
-    <child link="mount"/>
-    <origin xyz="0 0 0" rpy="0 0 -1.57"/>
-  </joint>
-  <link name="mount">
-    <visual>
-      <origin xyz="0 0 0.145" rpy="0 0 0"/>
-      <geometry>
-        <mesh filename="package://iiwa_tool_description/meshes/visual/mount.stl"/>
-      </geometry>
-      <material name="gray">
-        <color rgba="0.7 0.7 0.7 0.2"/>
-      </material>
-    </visual>
-    <collision>
-      <origin xyz="0 0 0.565" rpy="0 0 0"/>
-      <geometry>
-        <box size="0.25 0.25 0.82"/>
-      </geometry>
-    </collision>
-    <inertial>
-      <origin xyz="0 0 1" rpy="0 0 0"/>
-      <mass value="1"/>
-      <inertia
-        ixx="1.0" ixy="0.0" ixz="0.0"
-        iyy="1.0" iyz="0.0"
-        izz="1.0"/>
-    </inertial>
-  </link>
   <joint name="conveyor_joint" type="fixed">
-    <parent link="world"/>
+    <parent link="$(arg robot_name)_floating_link"/>
     <child link = "conveyor"/>
     <origin xyz="0.6 1.7 0" rpy="0 0 0"/>
@@ -104,7 +45,7 @@
   </link>
   <joint name="tv_joint" type="fixed">
-    <parent link="world"/>
+    <parent link="$(arg robot_name)_floating_link"/>
     <child link = "tv"/>
-    <origin xyz="0.6 -0.9 1.9" rpy="-0.1745 0 0.78"/>
+    <origin xyz="0.6 -0.5 1.9" rpy="-0.1745 0 0.78"/>
   </joint>
   <link name="tv">
@@ -134,5 +75,5 @@
   </link>
   <joint name="frame_joint" type="fixed">
-    <parent link="world"/>
+    <parent link="$(arg robot_name)_floating_link"/>
     <child link = "frame"/>
     <origin xyz="-0.2 0.8 0.84" rpy="0 0 0"/>
@@ -149,44 +90,66 @@
     </visual>
     <collision>
-      <origin xyz="0 0 -0.4" rpy="0 0 0"/>
-      <geometry>
-        <box size="1.0 1.0 0.7"/>
-      </geometry>
-    </collision>
-    <inertial>
-      <origin xyz="0 0 1" rpy="0 0 0"/>
-      <mass value="1"/>
-      <inertia
-        ixx="1.0" ixy="0.0" ixz="0.0"
-        iyy="1.0" iyz="0.0"
-        izz="1.0"/>
-    </inertial>
-  </link>
-  <joint name="workspace_mount_joint" type="fixed">
-      <origin xyz="0.30 0.34 0.016" rpy="0 0 0"/>
-      <parent link="frame"/>
-      <child link="workspace_mount"/>
-  </joint>
-  <link name="workspace_mount">
-      <visual>
-          <origin xyz="0 0 0" rpy="0 0 0"/>
-          <geometry>
-              <box size="0.3 0.3 0.03"/>
-          </geometry>
-          <material name="gray">
-              <color rgba="0.7 0.7 0.7 0.2"/>
-          </material>
-      </visual>
-      <collision>
-          <origin xyz="0 0 0" rpy="0 0 0"/>
-          <geometry>
-              <box size="0.3 0.3 0.03"/>
-          </geometry>
-      </collision>
-  </link>
+      <origin xyz="0 0 -0.5" rpy="0 0 0"/>
+      <geometry>
+        <box size="1.0 1.0 0.8"/>
+      </geometry>
+    </collision>
+    <inertial>
+      <origin xyz="0 0 1" rpy="0 0 0"/>
+      <mass value="1"/>
+      <inertia
+        ixx="1.0" ixy="0.0" ixz="0.0"
+        iyy="1.0" iyz="0.0"
+        izz="1.0"/>
+    </inertial>
+  </link>
+  <link name="workspace_mount1">
+    <visual>
+      <origin xyz="0 0 0" rpy="0 0 0"/>
+      <geometry>
+        <box size="0.3 0.3 0.03"/>
+      </geometry>
+      <material name="gray">
+        <color rgba="0.7 0.7 0.7 0.2"/>
+      </material>
+    </visual>
+    <collision>
+      <origin xyz="0 0 0" rpy="0 0 0"/>
+      <geometry>
+        <box size="0.3 0.3 0.03"/>
+      </geometry>
+    </collision>
+  </link>
+  <joint name="workspace_mount1_joint" type="fixed">
+    <origin xyz="0.1 0.5 0.85" rpy="0 0 3.14"/>
+    <parent link="$(arg robot_name)_floating_link"/>
+    <child link="workspace_mount1"/>
+  </joint>
+  <link name="workspace_mount2">
+    <visual>
+      <origin xyz="0 0 0" rpy="0 0 0"/>
+      <geometry>
+        <box size="0.3 0.3 0.03"/>
+      </geometry>
+      <material name="gray">
+        <color rgba="0.7 0.7 0.7 0.2"/>
+      </material>
+    </visual>
+    <collision>
+      <origin xyz="0 0 0" rpy="0 0 0"/>
+      <geometry>
+        <box size="0.3 0.3 0.03"/>
+      </geometry>
+    </collision>
+  </link>
+  <joint name="workspace_mount2_joint" type="fixed">
+    <origin xyz="-0.5 0.5 0.85" rpy="0 0 3.14"/>
+    <parent link="$(arg robot_name)_floating_link"/>
+    <child link="workspace_mount2"/>
+  </joint>
   <joint name="iiwa2_joint" type="fixed">
-    <parent link="workspace_mount"/>
+    <parent link="workspace_mount2"/>
     <child link = "iiwa2"/>
-    <origin xyz="0 0 0" rpy="1.57 0 0.785398"/>
+    <origin xyz="0 0 0" rpy="1.57 0 -2.37"/>
   </joint>
   <link name="iiwa2">
@@ -218,5 +181,5 @@
     <parent link="frame"/>
     <child link = "softjig"/>
-    <origin xyz="0.45 0 0" rpy="1.57 0 3.14"/>
+    <origin xyz="0.45 0.5 0" rpy="1.57 0 3.14"/>
   </joint>
   <link name="softjig">
@@ -226,5 +189,5 @@
         <mesh filename="package://iiwa_tool_description/meshes/visual/softjig.stl"/>
       </geometry>
-      <material name="dark_gray">
+      <material name="gray_dark">
         <color rgba="0.7 0.7 0.7 1.0"/>
       </material>
@@ -246,7 +209,7 @@
   </link>
   <joint name="round_table_joint" type="fixed">
-    <parent link="world"/>
+    <parent link="$(arg robot_name)_floating_link"/>
     <child link = "round_table"/>
-    <origin xyz="0 -0.7 0.55" rpy="0 0 0"/>
+    <origin xyz="0 -0.35 0.55" rpy="0 0 0"/>
   </joint>
   <link name="round_table">
@@ -306,6 +269,6 @@
   </link>
   <!-- Here we insert an iiwa14 robot in the scene, it's origin is just on top of the box previously defined. You can use 0,0,0 if you don't have that. -->
-  <xacro:iiwa14 hardware_interface="$(arg hardware_interface)" robot_name="$(arg robot_name)" parent="mount">
-    <origin xyz="0 0 0.972" rpy="0 0 -1.57"/>
+  <xacro:iiwa14 hardware_interface="$(arg hardware_interface)" robot_name="$(arg robot_name)" parent="workspace_mount1">
+    <origin xyz="0 0 0.016" rpy="0 0 2.36"/>
   </xacro:iiwa14>
   <!-- Add the gripper. Called from the file imported at the top of this code.-->
